File: pmod-io.kicad_pcb (KiCad board)
At the start: 4 copper layers, 50 x 30 mm, 55 parts, among them J1 PMOD, J2 430451628, U1 SN74LVC1G16DBVR, U2 SN74LVC1G16DBVR, U3 SN74LVC1G16DBVR, U4 SN74LVC1G16DBVR, U5 SN74AC14PWR, U6 SN74LVC3G34DCT, U7 SN74LVC3G34DCT, U8 SN74LVC3G34DCT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

Commit message: Passed DRC, ready to build?
Parts:
- moved H1 84.6 mm to (116.6, 85.0)
- moved R4 11.8 mm to (126.5, 77.2), turned to 90 degrees
- moved R2 11.8 mm to (126.5, 72.8), turned to 90 degrees
- moved R28 6.73 mm to (135.8, 96.2), turned to 90 degrees
- moved R25 6.64 mm to (135.8, 91.5), turned to 90 degrees
- moved R22 6.56 mm to (135.8, 86.8), turned to 90 degrees
- moved R19 6.49 mm to (135.8, 82.0), turned to 90 degrees
- moved R9 4.81 mm to (122.8, 73.8)
- moved R10 4.81 mm to (122.8, 71.8)
- moved R14 4.69 mm to (122.8, 76.2)
- moved C3 4.53 mm to (118.0, 77.2)
- moved U3 4.53 mm to (118.0, 77.2), turned to 180 degrees
- moved C1 4.51 mm to (118.0, 72.8)
- moved U1 4.51 mm to (118.0, 72.8), turned to 180 degrees
- moved R13 4.19 mm to (122.8, 78.2)
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Routing:
- net +3.3V: track 3.54 -> 56.5 mm, vias 4 -> 10
- net GND: track 1.52 -> 44.4 mm, vias 2 -> 10
- net /IN3: track 0.00 -> 25.8 mm
- net /PMOD_IN4: track 5.17 -> 30.2 mm
- net /IN1: track 0.00 -> 24.1 mm
- net /PMOD_IN2: track 10.3 -> 30.9 mm
- net Net-(U5-4Y): track 0.00 -> 20.0 mm
- net Net-(U5-5Y): track 0.00 -> 18.2 mm
- net Net-(U5-2Y): track 0.00 -> 16.7 mm
- net /OUT1: track 0.00 -> 16.1 mm
- net /PMOD_OUT4: track 11.5 -> 26.5 mm
- net /OUT2: track 0.00 -> 14.5 mm
- net Net-(U5-3Y): track 0.00 -> 14.3 mm
- net Net-(U9-3Y): track 0.00 -> 14.3 mm
- net /OUT4: track 0.00 -> 14.2 mm
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Other:
- board size 50 x 30 mm -> 47.2 x 30 mm
- board text added: "PMOD-IO V1.0 2025"
- board text removed: "PMOD-IO V1.0 10/2025"
