File: ttl-io.kicad_sch (KiCad schematic)
At the start: 56 parts, among them J1 PMOD, J2 430451628, U1 SN74LVC1G16DBVR, U2 SN74LVC1G16DBVR, U3 SN74LVC1G16DBVR, U4 SN74LVC1G16DBVR, U5 SN74AC14PWR, U6 SN74LVC3G34DCT, U7 SN74LVC3G34DCT, U8 SN74LVC3G34DCT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

Commit message: Updated part values/#s
Parts:
- R10, R12, R14, R16: value 50k -> 49.9k; Digikey 311-10.0KHRCT-ND -> 13-RC0603FR-1349K9LTR-ND; MPN RC0603FR-0710KL -> RC0603FR-1349K9L
- R11, R13, R15, R9: Digikey 311-10.0KHRCT-ND -> YAG1294TR-ND; MPN RC0603FR-0710KL -> RC0603FR-071KP
- R17, R18, R19, R20, R21, R22, R23, R24, R25, R26, R27, R28: value 143 -> 10; Digikey 311-1.00KCRTR-ND -> 13-RC0603FR-1310RLTR-ND; MPN RC0603FR-071KL -> RC0603FR-1310RL
- R29: Digikey 311-1.00KCRTR-ND -> YAG1294TR-ND; MPN RC0603FR-071KL -> RC0603FR-071KP
- U6, U7, U8, U9: MPN SN74LVC3G34DCUR -> SN74LVC3G34DCTR

Commit message: Updated sch notes and part info, ready for fab
Parts:
- removed TP1, TP2: TestPoint, 0local:TestPoint_Loop_D1.80mm_Drill1.0mm_Beaded, symbol 0local:TestPoint
- added TP1: TestPointRed, 0local:TestPoint_Loop_D1.80mm_Drill1.0mm_Beaded, symbol 0local:TestPointRed
- added TP2: TestPointBlack, 0local:TestPoint_Loop_D1.80mm_Drill1.0mm_Beaded, symbol 0local:TestPointBlack
- D1: Digikey 754-1116 -> 754-1116-2-ND
- H1: now left out of the parts list
- renumbered R11 to R10, R13 to R11, R15 to R12, R10 to R13, R12 to R14, R14 to R15
Connections:
- net +3.3V: now also TP1.1
- net GND: now also TP2.1
Other:
- note added: "10k pull-ups not needed for TXS0108E on carrier (due to internal pull-ups)"
- note added: "1k current limiting for higher voltage protection, 49.9k pull-down"
- note added: "3 parallel buffers for 50 ohm drive (3.3V/50 = 66mA)"
- note added: "50 ohm Termination Type R = 10: Far-End R = 143: Series or Double-Ended"
- note added: "Schmitt-Trigger for sharp edge from TXS0108E to drive 3 parallel gates each, and inverting for zero output during FPGA startup"
- note added: "Schmitt-Trigger for sharp edge, Open-Drain for TXS0108E, LVC for 6.5V input tolerance, and inverting for consitency with output"
- note removed: "3 parallel buffers for 50 ohm drive (3.3V/47 = 70mA)"
- note removed: "Schmitt-Trigger for sharp edge and Open-Drain for TXS0108E LVC for 6.5V input tolerance"
- note removed: "Schmitt-Trigger for sharp edge from TXS0108E to drive 3 gates simultaneously"
- note removed: "Termination Type R=143: Series or Double-Ended R=0: Far-End"
