File: ttl-io.kicad_sch (KiCad schematic)
At the start: 56 parts, among them J1 PMOD, J2 430451628, U1 SN74LVC1G16DBVR, U2 SN74LVC1G16DBVR, U3 SN74LVC1G16DBVR, U4 SN74LVC1G16DBVR, U5 SN74AC14PWR, U6 SN74LVC3G34DCT, U7 SN74LVC3G34DCT, U8 SN74LVC3G34DCT, U9 SN74LVC3G34DCT

Commit message: add title and copyright/license
adjust PCB page size to US letter
Other:
- company: (none) -> SPDX-FileCopyrightText: 2025 Osprey DCS
- title: (none) -> LVTTL PMOD
Changed lines of the file:
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@@
 	(generator_version "9.0")
 	(paper "A4")
+	(title_block
+		(title "LVTTL PMOD")
+		(company "SPDX-FileCopyrightText: 2025 Osprey DCS")
+		(comment 1 "SPDX-License-Identifier: CERN-OHL-S-2.0+")
+	)
 	(text "Schmitt-Trigger for sharp edge\nfrom TXS0108E to drive 3 parallel\ngates each, and inverting for zero\noutput during FPGA startup"
 		(exclude_from_sim no)
@@
 	(symbol
 		(lib_id "Graphic:Logo_Open_Hardware_Small")
-		(at 185.42 173.99 0)
+		(at 274.32 175.26 0)
 		(unit 1)
 		(exclude_from_sim yes)
@@
 		(fields_autoplaced yes)
 		(property "Reference" "Logo1"
-			(at 185.42 167.005 0)
+			(at 274.32 168.275 0)
 			(effects
 				(font
@@
 		)
 		(property "Value" "Logo_Open_Hardware_Small"
-			(at 185.42 179.705 0)
+			(at 274.32 180.975 0)
 			(effects
 				(font
@@
 		)
 		(property "Footprint" "0local:Logo_2X"
-			(at 185.42 173.99 0)
+			(at 274.32 175.26 0)
 			(effects
 				(font
@@
 		)
 		(property "Datasheet" "~"
-			(at 185.42 173.99 0)
+			(at 274.32 175.26 0)
 			(effects
 				(font
@@
 		)
 		(property "Description" "Open Hardware logo, small"
-			(at 185.42 173.99 0)
+			(at 274.32 175.26 0)
 			(effects
 				(font
@@
 		)
 		(property "MPN" "DNI"
-			(at 185.42 173.99 0)
+			(at 274.32 175.26 0)
 			(effects
 				(font

Commit message: 30x35mm version initial commit
Parts:
- removed J2: 430451628, 0local:430451628, symbol 0local:430451628
- added I1, I2, I3, I4, O1, O2, O3, O4: MMCX, 0local:MMCX_THT_Vertical, symbol 0local:MMCX
- renumbered C6 to C5, C7 to C6, C8 to C7, C9 to C8, C5 to C9, R5 to R1, R21 to R10, R25 to R11, R23 to R12, R24 to R13, R28 to R14, R26 to R15, R27 to R16, R13 to R17, R14 to R18, R15 to R19, R6 to R2, R16 to R20, R9 to R21, R10 to R22, R11 to R23, R12 to R24, R1 to R25, R2 to R26, R3 to R27, R4 to R28, R7 to R3, R8 to R4, R19 to R5, R17 to R6, R18 to R7, R22 to R8, R20 to R9, U5 to U1, U6 to U2, U7 to U3, U8 to U4, U9 to U5, U1 to U6, U2 to U7, U3 to U8, U4 to U9
Connections:
- net +3.3V: now also U1.3 (2A); no longer U1.1 (1A)
- net GND: now also I1.2 (Ext), I2.2 (Ext), I3.2 (Ext), I4.2 (Ext), O1.2 (Ext), O2.2 (Ext), O3.2 (Ext), O4.2 (Ext)
- net IN1: now also I1.1 (In)
- net IN2: now also I2.1 (In)
- net IN3: now also I3.1 (In)
- net IN4: now also I4.1 (In)
- net OUT1: now also O1.1 (In)
- net OUT2: now also O2.1 (In)
- net OUT3: now also O3.1 (In)
- net OUT4: now also O4.1 (In)
- net PMOD_OUT1: now also U1.11 (5A); no longer U1.9 (4A)
- net PMOD_OUT2: now also U1.9 (4A); no longer U1.11 (5A)
- net PMOD_OUT3: now also U1.5 (3A); no longer U1.3 (2A)
- net PMOD_OUT4: now also U1.1 (1A); no longer U1.5 (3A)
- net at U2.1 (1A), U2.3 (2A), U2.6 (3A): now also U1.10 (5Y); no longer U1.8 (4Y)
- net at U3.1 (1A), U3.3 (2A), U3.6 (3A): now also U1.8 (4Y); no longer U1.10 (5Y)
- net at U4.1 (1A), U4.3 (2A), U4.6 (3A): now also U1.6 (3Y); no longer U1.4 (2Y)
- net at U1.2 (1Y): now also U5.1 (1A), U5.3 (2A), U5.6 (3A)
Other:
- moved on the sheet: C10, C11, C9, D1, H1, J1, R1, R11, R12, R14, R15, R2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

Commit message: slotted mounting hole
Parts:
- removed Logo1: Logo_Open_Hardware_Small, 0local:Logo_2X, symbol Graphic:Logo_Open_Hardware_Small
Changed lines of the file:
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@@
-	)
-	(symbol
-		(lib_id "Graphic:Logo_Open_Hardware_Small")
-		(at 274.32 175.26 0)
-		(unit 1)
-		(exclude_from_sim yes)
-		(in_bom no)
-		(on_board yes)
-		(dnp no)
-		(fields_autoplaced yes)
-		(property "Reference" "Logo1"
-			(at 274.32 168.275 0)
-			(effects
-				(font
-					(size 1.27 1.27)
-				)
-				(hide yes)
-			)
-		)
-		(property "Value" "Logo_Open_Hardware_Small"
-			(at 274.32 180.975 0)
-			(effects
-				(font
-					(size 1.27 1.27)
-				)
-				(hide yes)
-			)
-		)
-		(property "Footprint" "0local:Logo_2X"
-			(at 274.32 175.26 0)
-			(effects
-				(font
-					(size 1.27 1.27)
-				)
-				(hide yes)
-			)
-		)
-		(property "Datasheet" "~"
-			(at 274.32 175.26 0)
-			(effects
-				(font
-					(size 1.27 1.27)
-				)
-				(hide yes)
-			)
-		)
-		(property "Description" "Open Hardware logo, small"
-			(at 274.32 175.26 0)
-			(effects
-				(font
-					(size 1.27 1.27)
-				)
-				(hide yes)
-			)
-		)
-		(property "MPN" "DNI"
-			(at 274.32 175.26 0)
-			(effects
-				(font
-					(size 1.27 1.27)
-				)
-				(hide yes)
-			)
-		)
-		(instances
-			(project "ttl-io"
-				(path "/c58eba57-e11a-4091-8cda-9e71ea4f3e44"
-					(reference "Logo1")
-					(unit 1)
-				)
-			)
-		)
 	)
 	(symbol

Commit message: Updated 0805 resistor part #
Parts:
- R10, R11, R12, R13, R14, R15, R16, R5, R6, R7, R8, R9: Digikey 13-RC0603FR-1310RLTR-ND -> 13-RC0805FR-1310RLTR-ND; MPN RC0603FR-1310RL -> RC0805FR-1310RL
Changed lines of the file:
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@@
 	(title_block
 		(title "LVTTL PMOD")
-		(date "2025-11-04")
+		(date "2025-11-12")
 		(rev "v1.0")
 		(company "SPDX-FileCopyrightText: 2025 Osprey DCS")
@@
 			)
 		)
-		(property "Description" "10 Ohms ±1% 0.1W, 1/10W Chip Resistor 0603 (1608 Metric) Moisture Resistant Thick Film"
+		(property "Description" "10 Ohms ±1% 0.125W, 1/8W Chip Resistor 0805 (2012 Metric) Moisture Resistant Thick Film"
 			(at 162.56 92.71 0)
 			(effects
@@
 			)
 		)
-		(property "Digikey" "13-RC0603FR-1310RLTR-ND"
+		(property "Digikey" "13-RC0805FR-1310RLTR-ND"
 			(at 162.56 92.71 90)
 			(effects
@@
 			)
 		)
-		(property "MPN" "RC0603FR-1310RL"
+		(property "MPN" "RC0805FR-1310RL"
 			(at 162.56 92.71 90)
 			(effects
@@
 			)
 		)
-		(property "Description" "10 Ohms ±1% 0.1W, 1/10W Chip Resistor 0603 (1608 Metric) Moisture Resistant Thick Film"
+		(property "Description" "10 Ohms ±1% 0.125W, 1/8W Chip Resistor 0805 (2012 Metric) Moisture Resistant Thick Film"
 			(at 162.56 101.6 0)
 			(effects
@@
 			)
 		)
-		(property "Digikey" "13-RC0603FR-1310RLTR-ND"
+		(property "Digikey" "13-RC0805FR-1310RLTR-ND"
 			(at 162.56 101.6 90)
 			(effects
@@
 			)
 		)
-		(property "MPN" "RC0603FR-1310RL"
+		(property "MPN" "RC0805FR-1310RL"
 			(at 162.56 101.6 90)
 			(effects
@@
 			)
 		)
-		(property "Description" "10 Ohms ±1% 0.1W, 1/10W Chip Resistor 0603 (1608 Metric) Moisture Resistant Thick Film"
+		(property "Description" "10 Ohms ±1% 0.125W, 1/8W Chip Resistor 0805 (2012 Metric) Moisture Resistant Thick Film"
 			(at 250.19 107.95 0)
 			(effects
@@
 			)
 		)
-		(property "Digikey" "13-RC0603FR-1310RLTR-ND"
+		(property "Digikey" "13-RC0805FR-1310RLTR-ND"
 			(at 250.19 107.95 90)
 			(effects
@@
 			)
 		)
-		(property "MPN" "RC0603FR-1310RL"
+		(property "MPN" "RC0805FR-1310RL"
 			(at 250.19 107.95 90)
 			(effects
@@
 			)
 		)
-		(property "Description" "10 Ohms ±1% 0.1W, 1/10W Chip Resistor 0603 (1608 Metric) Moisture Resistant Thick Film"
+		(property "Description" "10 Ohms ±1% 0.125W, 1/8W Chip Resistor 0805 (2012 Metric) Moisture Resistant Thick Film"
 			(at 250.19 116.84 0)
 			(effects
@@
 			)
 		)
-		(property "Digikey" "13-RC0603FR-1310RLTR-ND"
+		(property "Digikey" "13-RC0805FR-1310RLTR-ND"
 			(at 250.19 116.84 90)
 			(effects
@@
 			)
 		)
-		(property "MPN" "RC0603FR-1310RL"
+		(property "MPN" "RC0805FR-1310RL"
 			(at 250.19 116.84 90)
 			(effects
@@
 			)
 		)
-		(property "Description" "10 Ohms ±1% 0.1W, 1/10W Chip Resistor 0603 (1608 Metric) Moisture Resistant Thick Film"
+		(property "Description" "10 Ohms ±1% 0.125W, 1/8W Chip Resistor 0805 (2012 Metric) Moisture Resistant Thick Film"
 			(at 162.56 143.51 0)
 			(effects
@@
 			)
 		)
-		(property "Digikey" "13-RC0603FR-1310RLTR-ND"
+		(property "Digikey" "13-RC0805FR-1310RLTR-ND"
 			(at 162.56 143.51 90)
 			(effects
@@
 			)
 		)
-		(property "MPN" "RC0603FR-1310RL"
+		(property "MPN" "RC0805FR-1310RL"
 			(at 162.56 143.51 90)
 			(effects
@@
 			)
 		)
-		(property "Description" "10 Ohms ±1% 0.1W, 1/10W Chip Resistor 0603 (1608 Metric) Moisture Resistant Thick Film"
+		(property "Description" "10 Ohms ±1% 0.125W, 1/8W Chip Resistor 0805 (2012 Metric) Moisture Resistant Thick Film"
 			(at 250.19 149.86 0)
 			(effects
@@
 			)
 		)
-		(property "Digikey" "13-RC0603FR-1310RLTR-ND"
+		(property "Digikey" "13-RC0805FR-1310RLTR-ND"
 			(at 250.19 149.86 90)
 			(effects
@@
 			)
 		)
-		(property "MPN" "RC0603FR-1310RL"
+		(property "MPN" "RC0805FR-1310RL"
 			(at 250.19 149.86 90)
 			(effects
@@
 			)
 		)
-		(property "Description" "10 Ohms ±1% 0.1W, 1/10W Chip Resistor 0603 (1608 Metric) Moisture Resistant Thick Film"
+		(property "Description" "10 Ohms ±1% 0.125W, 1/8W Chip Resistor 0805 (2012 Metric) Moisture Resistant Thick Film"
 			(at 250.19 140.97 0)
 			(effects
@@
 			)
 		)
-		(property "Digikey" "13-RC0603FR-1310RLTR-ND"
+		(property "Digikey" "13-RC0805FR-1310RLTR-ND"
 			(at 250.19 140.97 90)
 			(effects
@@
 			)
 		)
-		(property "MPN" "RC0603FR-1310RL"
+		(property "MPN" "RC0805FR-1310RL"
 			(at 250.19 140.97 90)
 			(effects
@@
 			)
 		)
-		(property "Description" "10 Ohms ±1% 0.1W, 1/10W Chip Resistor 0603 (1608 Metric) Moisture Resistant Thick Film"
+		(property "Description" "10 Ohms ±1% 0.125W, 1/8W Chip Resistor 0805 (2012 Metric) Moisture Resistant Thick Film"
 			(at 162.56 125.73 0)
 			(effects
@@
 			)
 		)
-		(property "Digikey" "13-RC0603FR-1310RLTR-ND"
+		(property "Digikey" "13-RC0805FR-1310RLTR-ND"
 			(at 162.56 125.73 90)
 			(effects
@@
 			)
 		)
-		(property "MPN" "RC0603FR-1310RL"
+		(property "MPN" "RC0805FR-1310RL"
 			(at 162.56 125.73 90)
 			(effects
@@
 			)
 		)
-		(property "Description" "10 Ohms ±1% 0.1W, 1/10W Chip Resistor 0603 (1608 Metric) Moisture Resistant Thick Film"
+		(property "Description" "10 Ohms ±1% 0.125W, 1/8W Chip Resistor 0805 (2012 Metric) Moisture Resistant Thick Film"
 			(at 250.19 158.75 0)
 			(effects
@@
 			)
 		)
-		(property "Digikey" "13-RC0603FR-1310RLTR-ND"
+		(property "Digikey" "13-RC0805FR-1310RLTR-ND"
 			(at 250.19 158.75 90)
 			(effects
@@
 			)
 		)
-		(property "MPN" "RC0603FR-1310RL"
+		(property "MPN" "RC0805FR-1310RL"
 			(at 250.19 158.75 90)
 			(effects
@@
 			)
 		)
-		(property "Description" "10 Ohms ±1% 0.1W, 1/10W Chip Resistor 0603 (1608 Metric) Moisture Resistant Thick Film"
+		(property "Description" "10 Ohms ±1% 0.125W, 1/8W Chip Resistor 0805 (2012 Metric) Moisture Resistant Thick Film"
 			(at 162.56 110.49 0)
 			(effects
@@
 			)
 		)
-		(property "Digikey" "13-RC0603FR-1310RLTR-ND"
+		(property "Digikey" "13-RC0805FR-1310RLTR-ND"
 			(at 162.56 110.49 90)
 			(effects
@@
 			)
 		)
-		(property "MPN" "RC0603FR-1310RL"
+		(property "MPN" "RC0805FR-1310RL"
 			(at 162.56 110.49 90)
 			(effects
@@
 			)
 		)
-		(property "Description" "10 Ohms ±1% 0.1W, 1/10W Chip Resistor 0603 (1608 Metric) Moisture Resistant Thick Film"
+		(property "Description" "10 Ohms ±1% 0.125W, 1/8W Chip Resistor 0805 (2012 Metric) Moisture Resistant Thick Film"
 			(at 162.56 134.62 0)
 			(effects
@@
 			)
 		)
-		(property "Digikey" "13-RC0603FR-1310RLTR-ND"
+		(property "Digikey" "13-RC0805FR-1310RLTR-ND"
 			(at 162.56 134.62 90)
 			(effects
@@
 			)
 		)
-		(property "MPN" "RC0603FR-1310RL"
+		(property "MPN" "RC0805FR-1310RL"
 			(at 162.56 134.62 90)
 			(effects
@@
 			)
 		)
-		(property "Description" "10 Ohms ±1% 0.1W, 1/10W Chip Resistor 0603 (1608 Metric) Moisture Resistant Thick Film"
+		(property "Description" "10 Ohms ±1% 0.125W, 1/8W Chip Resistor 0805 (2012 Metric) Moisture Resistant Thick Film"
 			(at 250.19 125.73 0)
 			(effects
@@
 			)
 		)
-		(property "Digikey" "13-RC0603FR-1310RLTR-ND"
+		(property "Digikey" "13-RC0805FR-1310RLTR-ND"
 			(at 250.19 125.73 90)
 			(effects
@@
 			)
 		)
-		(property "MPN" "RC0603FR-1310RL"
+		(property "MPN" "RC0805FR-1310RL"
 			(at 250.19 125.73 90)
 			(effects

Commit message: Fixed 10 ohm res part #
Parts:
- R10, R11, R12, R13, R14, R15, R16, R5, R6, R7, R8, R9: Digikey 13-RC0805FR-1310RLTR-ND -> 13-RC0805FR-1010RLTR-ND; MPN RC0805FR-1310RL -> RC0805FR-1010RL
Changed lines of the file:
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@@
 			)
 		)
-		(property "Digikey" "13-RC0805FR-1310RLTR-ND"
+		(property "Digikey" "13-RC0805FR-1010RLTR-ND"
 			(at 162.56 92.71 90)
 			(effects
@@
 			)
 		)
-		(property "MPN" "RC0805FR-1310RL"
+		(property "MPN" "RC0805FR-1010RL"
 			(at 162.56 92.71 90)
 			(effects
@@
 			)
 		)
-		(property "Digikey" "13-RC0805FR-1310RLTR-ND"
+		(property "Digikey" "13-RC0805FR-1010RLTR-ND"
 			(at 162.56 101.6 90)
 			(effects
@@
 			)
 		)
-		(property "MPN" "RC0805FR-1310RL"
+		(property "MPN" "RC0805FR-1010RL"
 			(at 162.56 101.6 90)
 			(effects
@@
 			)
 		)
-		(property "Digikey" "13-RC0805FR-1310RLTR-ND"
+		(property "Digikey" "13-RC0805FR-1010RLTR-ND"
 			(at 250.19 107.95 90)
 			(effects
@@
 			)
 		)
-		(property "MPN" "RC0805FR-1310RL"
+		(property "MPN" "RC0805FR-1010RL"
 			(at 250.19 107.95 90)
 			(effects
@@
 			)
 		)
-		(property "Digikey" "13-RC0805FR-1310RLTR-ND"
+		(property "Digikey" "13-RC0805FR-1010RLTR-ND"
 			(at 250.19 116.84 90)
 			(effects
@@
 			)
 		)
-		(property "MPN" "RC0805FR-1310RL"
+		(property "MPN" "RC0805FR-1010RL"
 			(at 250.19 116.84 90)
 			(effects
@@
 			)
 		)
-		(property "Digikey" "13-RC0805FR-1310RLTR-ND"
+		(property "Digikey" "13-RC0805FR-1010RLTR-ND"
 			(at 162.56 143.51 90)
 			(effects
@@
 			)
 		)
-		(property "MPN" "RC0805FR-1310RL"
+		(property "MPN" "RC0805FR-1010RL"
 			(at 162.56 143.51 90)
 			(effects
@@
 			)
 		)
-		(property "Digikey" "13-RC0805FR-1310RLTR-ND"
+		(property "Digikey" "13-RC0805FR-1010RLTR-ND"
 			(at 250.19 149.86 90)
 			(effects
@@
 			)
 		)
-		(property "MPN" "RC0805FR-1310RL"
+		(property "MPN" "RC0805FR-1010RL"
 			(at 250.19 149.86 90)
 			(effects
@@
 			)
 		)
-		(property "Digikey" "13-RC0805FR-1310RLTR-ND"
+		(property "Digikey" "13-RC0805FR-1010RLTR-ND"
 			(at 250.19 140.97 90)
 			(effects
@@
 			)
 		)
-		(property "MPN" "RC0805FR-1310RL"
+		(property "MPN" "RC0805FR-1010RL"
 			(at 250.19 140.97 90)
 			(effects
@@
 			)
 		)
-		(property "Digikey" "13-RC0805FR-1310RLTR-ND"
+		(property "Digikey" "13-RC0805FR-1010RLTR-ND"
 			(at 162.56 125.73 90)
 			(effects
@@
 			)
 		)
-		(property "MPN" "RC0805FR-1310RL"
+		(property "MPN" "RC0805FR-1010RL"
 			(at 162.56 125.73 90)
 			(effects
@@
 			)
 		)
-		(property "Digikey" "13-RC0805FR-1310RLTR-ND"
+		(property "Digikey" "13-RC0805FR-1010RLTR-ND"
 			(at 250.19 158.75 90)
 			(effects
@@
 			)
 		)
-		(property "MPN" "RC0805FR-1310RL"
+		(property "MPN" "RC0805FR-1010RL"
 			(at 250.19 158.75 90)
 			(effects
@@
 			)
 		)
-		(property "Digikey" "13-RC0805FR-1310RLTR-ND"
+		(property "Digikey" "13-RC0805FR-1010RLTR-ND"
 			(at 162.56 110.49 90)
 			(effects
@@
 			)
 		)
-		(property "MPN" "RC0805FR-1310RL"
+		(property "MPN" "RC0805FR-1010RL"
 			(at 162.56 110.49 90)
 			(effects
@@
 			)
 		)
-		(property "Digikey" "13-RC0805FR-1310RLTR-ND"
+		(property "Digikey" "13-RC0805FR-1010RLTR-ND"
 			(at 162.56 134.62 90)
 			(effects
@@
 			)
 		)
-		(property "MPN" "RC0805FR-1310RL"
+		(property "MPN" "RC0805FR-1010RL"
 			(at 162.56 134.62 90)
 			(effects
@@
 			)
 		)
-		(property "Digikey" "13-RC0805FR-1310RLTR-ND"
+		(property "Digikey" "13-RC0805FR-1010RLTR-ND"
 			(at 250.19 125.73 90)
 			(effects
@@
 			)
 		)
-		(property "MPN" "RC0805FR-1310RL"
+		(property "MPN" "RC0805FR-1010RL"
 			(at 250.19 125.73 90)
 			(effects
