File: ttl-io.kicad_pcb (KiCad board)
At the start: 4 copper layers, 35 x 30 mm, 62 parts, among them J1 PMOD, U1 SN74AC14PWR, U2 SN74LVC3G34DCT, U3 SN74LVC3G34DCT, U4 SN74LVC3G34DCT, U5 SN74LVC3G34DCT, U6 SN74LVC1G16DBVR, U7 SN74LVC1G16DBVR, U8 SN74LVC1G16DBVR, U9 SN74LVC1G16DBVR

Commit message: add silkscreen bar under passives which should be placed
Parts:
- R1, R2, R25, R26, R27, R28, R3, R4: footprint 0local:R_0603_1608Metric -> 0local:R_0603_1608Metric_DNP
